File: ButterflyFC.brd (EAGLE design)
At the start: 38 x 36 mm, 7 parts

Commit message: Added labels for Butterfly pinout
Parts:
- renumbered JP1 to 13, JP2 to 12
Other:
- board text added: "VIN"
Changed lines of the file:
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@@
 <text x="16" y="29" size="1" layer="21">GND</text>
 <text x="50" y="21" size="1.4224" layer="21" font="fixed">1</text>
+<text x="31.127115625" y="11.8060125" size="1" layer="21" rot="R90">VIN</text>
+<text x="41.2118625" y="11.593903125" size="1" layer="21" rot="R90">GND</text>
 </plain>
 <attributes>
@@
 <element name="ESCMTR" library="pinhead" library_urn="urn:adsk.eagle:library:325" package="1X04" package3d_urn="urn:adsk.eagle:package:22407/2" value="" x="48.88" y="27.1" rot="R270"/>
 <element name="FRAME1" library="SparkFun-Aesthetics" library_urn="urn:adsk.eagle:library:507" package="CREATIVE_COMMONS" package3d_urn="urn:adsk.eagle:package:37121/1" value="FRAME-LETTER" x="12.99" y="-0.76"/>
-<element name="JP1" library="pinhead" library_urn="urn:adsk.eagle:library:325" package="1X09" package3d_urn="urn:adsk.eagle:package:22483/2" value="" x="28.21" y="23.29" rot="R270"/>
-<element name="JP2" library="pinhead" library_urn="urn:adsk.eagle:library:325" package="1X09" package3d_urn="urn:adsk.eagle:package:22483/2" value="" x="43.26" y="23.29" rot="R270"/>
+<element name="13" library="pinhead" library_urn="urn:adsk.eagle:library:325" package="1X09" package3d_urn="urn:adsk.eagle:package:22483/2" value="" x="28.21" y="23.29" rot="R270"/>
+<element name="12" library="pinhead" library_urn="urn:adsk.eagle:library:325" package="1X09" package3d_urn="urn:adsk.eagle:package:22483/2" value="" x="43.26" y="23.29" rot="R270"/>
 <element name="SBUS" library="pinhead" library_urn="urn:adsk.eagle:library:325" package="1X03" package3d_urn="urn:adsk.eagle:package:22458/2" value="" x="20.69" y="32.13" rot="R270"/>
 <element name="ESCPWR" library="pinhead" library_urn="urn:adsk.eagle:library:325" package="1X02" package3d_urn="urn:adsk.eagle:package:22435/2" value="" x="21.32" y="14.4" rot="R90"/>
@@
 <contactref element="SBUS" pad="3"/>
 <contactref element="DSM" pad="2"/>
-<contactref element="JP1" pad="8"/>
+<contactref element="13" pad="8"/>
 <contactref element="ESCPWR" pad="2"/>
 <wire x1="20.4912" y1="24.2448" x2="21.304" y2="23.432" width="0.2032" layer="1"/>
@@
 <signal name="VCC">
 <contactref element="SBUS" pad="2"/>
-<contactref element="JP1" pad="9"/>
+<contactref element="13" pad="9"/>
 <contactref element="ESCPWR" pad="1"/>
 <wire x1="28.0604" y1="13.0688" x2="28.21" y2="13.13" width="0.1524" layer="1"/>
@@
 </signal>
 <signal name="RX1">
-<contactref element="JP2" pad="8"/>
+<contactref element="12" pad="8"/>
 <contactref element="SBUS" pad="1"/>
 <contactref element="DSM" pad="3"/>
@@
 </signal>
 <signal name="N$3">
-<contactref element="JP2" pad="5"/>
+<contactref element="12" pad="5"/>
 <contactref element="ESCMTR" pad="4"/>
 <wire x1="43.3004" y1="23.2796" x2="43.26" y2="23.29" width="0.1524" layer="1"/>
@@
 <signal name="N$6">
 <contactref element="ESCMTR" pad="3"/>
-<contactref element="JP2" pad="4"/>
+<contactref element="12" pad="4"/>
 <wire x1="43.3004" y1="25.8704" x2="43.26" y2="25.83" width="0.1524" layer="1"/>
 <wire x1="48.736" y1="25.8704" x2="43.4528" y2="25.8704" width="0.2032" layer="1"/>
@@
 <signal name="N$2">
 <contactref element="ESCMTR" pad="1"/>
-<contactref element="JP2" pad="2"/>
+<contactref element="12" pad="2"/>
 <wire x1="43.3004" y1="30.8996" x2="43.26" y2="30.91" width="0.1524" layer="1"/>
 <wire x1="48.736" y1="30.9504" x2="43.4528" y2="30.9504" width="0.2032" layer="1"/>
@@
 <signal name="N$4">
 <contactref element="ESCMTR" pad="2"/>
-<contactref element="JP2" pad="3"/>
+<contactref element="12" pad="3"/>
 <wire x1="43.3004" y1="28.3088" x2="43.26" y2="28.37" width="0.1524" layer="1"/>
 <wire x1="48.736" y1="28.3088" x2="43.4528" y2="28.3088" width="0.2032" layer="1"/>
@@
 </signal>
 <signal name="3V3">
-<contactref element="JP1" pad="7"/>
+<contactref element="13" pad="7"/>
 <contactref element="DSM" pad="1"/>
 <wire x1="21.7424" y1="24.5872" x2="21.5392" y2="24.5872" width="0.2032" layer="1"/>

Commit message: Corrected labels on top pins
Parts:
- renumbered 12 to 7, 13 to A0
Changed lines of the file:
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@@
 <element name="ESCMTR" library="pinhead" library_urn="urn:adsk.eagle:library:325" package="1X04" package3d_urn="urn:adsk.eagle:package:22407/2" value="" x="48.88" y="27.1" rot="R270"/>
 <element name="FRAME1" library="SparkFun-Aesthetics" library_urn="urn:adsk.eagle:library:507" package="CREATIVE_COMMONS" package3d_urn="urn:adsk.eagle:package:37121/1" value="FRAME-LETTER" x="12.99" y="-0.76"/>
-<element name="13" library="pinhead" library_urn="urn:adsk.eagle:library:325" package="1X09" package3d_urn="urn:adsk.eagle:package:22483/2" value="" x="28.21" y="23.29" rot="R270"/>
-<element name="12" library="pinhead" library_urn="urn:adsk.eagle:library:325" package="1X09" package3d_urn="urn:adsk.eagle:package:22483/2" value="" x="43.26" y="23.29" rot="R270"/>
+<element name="A0" library="pinhead" library_urn="urn:adsk.eagle:library:325" package="1X09" package3d_urn="urn:adsk.eagle:package:22483/2" value="" x="28.21" y="23.29" rot="R270"/>
+<element name="7" library="pinhead" library_urn="urn:adsk.eagle:library:325" package="1X09" package3d_urn="urn:adsk.eagle:package:22483/2" value="" x="43.26" y="23.29" rot="R270"/>
 <element name="SBUS" library="pinhead" library_urn="urn:adsk.eagle:library:325" package="1X03" package3d_urn="urn:adsk.eagle:package:22458/2" value="" x="20.69" y="32.13" rot="R270"/>
 <element name="ESCPWR" library="pinhead" library_urn="urn:adsk.eagle:library:325" package="1X02" package3d_urn="urn:adsk.eagle:package:22435/2" value="" x="21.32" y="14.4" rot="R90"/>
@@
 <contactref element="SBUS" pad="3"/>
 <contactref element="DSM" pad="2"/>
-<contactref element="13" pad="8"/>
+<contactref element="A0" pad="8"/>
 <contactref element="ESCPWR" pad="2"/>
 <wire x1="20.4912" y1="24.2448" x2="21.304" y2="23.432" width="0.2032" layer="1"/>
@@
 <signal name="VCC">
 <contactref element="SBUS" pad="2"/>
-<contactref element="13" pad="9"/>
+<contactref element="A0" pad="9"/>
 <contactref element="ESCPWR" pad="1"/>
 <wire x1="28.0604" y1="13.0688" x2="28.21" y2="13.13" width="0.1524" layer="1"/>
@@
 </signal>
 <signal name="RX1">
-<contactref element="12" pad="8"/>
+<contactref element="7" pad="8"/>
 <contactref element="SBUS" pad="1"/>
 <contactref element="DSM" pad="3"/>
@@
 </signal>
 <signal name="N$3">
-<contactref element="12" pad="5"/>
+<contactref element="7" pad="5"/>
 <contactref element="ESCMTR" pad="4"/>
 <wire x1="43.3004" y1="23.2796" x2="43.26" y2="23.29" width="0.1524" layer="1"/>
@@
 <signal name="N$6">
 <contactref element="ESCMTR" pad="3"/>
-<contactref element="12" pad="4"/>
+<contactref element="7" pad="4"/>
 <wire x1="43.3004" y1="25.8704" x2="43.26" y2="25.83" width="0.1524" layer="1"/>
 <wire x1="48.736" y1="25.8704" x2="43.4528" y2="25.8704" width="0.2032" layer="1"/>
@@
 <signal name="N$2">
 <contactref element="ESCMTR" pad="1"/>
-<contactref element="12" pad="2"/>
+<contactref element="7" pad="2"/>
 <wire x1="43.3004" y1="30.8996" x2="43.26" y2="30.91" width="0.1524" layer="1"/>
 <wire x1="48.736" y1="30.9504" x2="43.4528" y2="30.9504" width="0.2032" layer="1"/>
@@
 <signal name="N$4">
 <contactref element="ESCMTR" pad="2"/>
-<contactref element="12" pad="3"/>
+<contactref element="7" pad="3"/>
 <wire x1="43.3004" y1="28.3088" x2="43.26" y2="28.37" width="0.1524" layer="1"/>
 <wire x1="48.736" y1="28.3088" x2="43.4528" y2="28.3088" width="0.2032" layer="1"/>
@@
 </signal>
 <signal name="3V3">
-<contactref element="13" pad="7"/>
+<contactref element="A0" pad="7"/>
 <contactref element="DSM" pad="1"/>
 <wire x1="21.7424" y1="24.5872" x2="21.5392" y2="24.5872" width="0.2032" layer="1"/>

Commit message: Goosed-up power-wire widths
Connections:
- net N$2 renamed MTR4
- net N$3 renamed MTR1
- net N$4 renamed MTR3
- net N$6 renamed MTR2
Changed lines of the file:
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@@
 <setting verticaltext="up"/>
 </settings>
-<grid distance="1" unitdist="mm" unit="mm" style="dots" multiple="1" display="yes" altdistance="5" altunitdist="mil" altunit="mil"/>
+<grid distance="39.3700787" unitdist="mil" unit="mil" style="dots" multiple="1" display="yes" altdistance="5" altunitdist="mil" altunit="mil"/>
 <layers>
 <layer number="1" name="Top" color="4" fill="1" visible="yes" active="yes"/>
@@
 <contactref element="A0" pad="8"/>
 <contactref element="ESCPWR" pad="2"/>
-<wire x1="20.4912" y1="24.2448" x2="21.304" y2="23.432" width="0.2032" layer="1"/>
-<wire x1="20.4912" y1="29.528" x2="20.4912" y2="24.2448" width="0.2032" layer="1"/>
+<wire x1="20.4912" y1="24.2448" x2="21.304" y2="23.432" width="0.254" layer="1"/>
+<wire x1="20.4912" y1="29.528" x2="20.4912" y2="24.2448" width="0.254" layer="1"/>
 <wire x1="21.304" y1="23.432" x2="21.5" y2="23.29" width="0.2032" layer="1"/>
 <wire x1="20.4912" y1="29.528" x2="20.69" y2="29.59" width="0.2032" layer="1"/>
-<wire x1="28.0096" y1="15.7104" x2="22.5232" y2="15.7104" width="0.2032" layer="1"/>
+<wire x1="28.0096" y1="15.7104" x2="22.5232" y2="15.7104" width="0.762" layer="1"/>
 <wire x1="22.5232" y1="15.7104" x2="21.5072" y2="15.7104" width="0.2032" layer="1"/>
 <wire x1="21.5072" y1="15.7104" x2="21.32" y2="15.67" width="0.2032" layer="1"/>
 <wire x1="28.0096" y1="15.7104" x2="28.21" y2="15.67" width="0.2032" layer="1"/>
-<wire x1="22.5232" y1="22.2128" x2="21.5072" y2="23.2288" width="0.2032" layer="1"/>
-<wire x1="22.5232" y1="15.7104" x2="22.5232" y2="22.2128" width="0.2032" layer="1"/>
+<wire x1="22.5232" y1="22.2128" x2="21.5072" y2="23.2288" width="0.254" layer="1"/>
+<wire x1="22.5232" y1="15.7104" x2="22.5232" y2="22.2128" width="0.254" layer="1"/>
 <wire x1="21.5072" y1="23.2288" x2="21.5" y2="23.29" width="0.2032" layer="1"/>
 <wire x1="22.5232" y1="15.7104" x2="21.32" y2="15.67" width="0.2032" layer="1"/>
@@
 <contactref element="ESCPWR" pad="1"/>
 <wire x1="28.0604" y1="13.0688" x2="28.21" y2="13.13" width="0.1524" layer="1"/>
-<wire x1="18.6624" y1="30.1376" x2="20.4912" y2="31.9664" width="0.2032" layer="1"/>
-<wire x1="18.6624" y1="15.9136" x2="18.6624" y2="30.1376" width="0.2032" layer="1"/>
-<wire x1="21.304" y1="13.272" x2="18.6624" y2="15.9136" width="0.2032" layer="1"/>
+<wire x1="18.6624" y1="30.1376" x2="20.4912" y2="31.9664" width="0.254" layer="1"/>
+<wire x1="18.6624" y1="15.9136" x2="18.6624" y2="30.1376" width="0.254" layer="1"/>
+<wire x1="21.304" y1="13.272" x2="18.6624" y2="15.9136" width="0.254" layer="1"/>
 <wire x1="20.4912" y1="31.9664" x2="20.69" y2="32.13" width="0.2032" layer="1"/>
 <wire x1="21.304" y1="13.272" x2="21.32" y2="13.13" width="0.2032" layer="1"/>
-<wire x1="21.5072" y1="13.0688" x2="28.0096" y2="13.0688" width="0.2032" layer="1"/>
+<wire x1="21.5072" y1="13.0688" x2="28.0096" y2="13.0688" width="0.762" layer="1"/>
 <wire x1="28.0096" y1="13.0688" x2="28.21" y2="13.13" width="0.2032" layer="1"/>
 <wire x1="21.5072" y1="13.0688" x2="21.32" y2="13.13" width="0.2032" layer="1"/>
@@
 <contactref element="DSM" pad="3"/>
 <wire x1="43.148" y1="15.812" x2="43.26" y2="15.67" width="0.1524" layer="16"/>
-<wire x1="22.7264" y1="23.0256" x2="21.5072" y2="21.8064" width="0.2032" layer="16"/>
+<wire x1="22.7264" y1="23.0256" x2="21.5072" y2="21.8064" width="0.254" layer="16"/>
 <wire x1="22.7264" y1="32.576" x2="22.7264" y2="23.0256" width="0.2032" layer="16"/>
-<wire x1="20.6944" y1="34.608" x2="22.7264" y2="32.576" width="0.2032" layer="16"/>
+<wire x1="20.6944" y1="34.608" x2="22.7264" y2="32.576" width="0.254" layer="16"/>
 <wire x1="21.5072" y1="21.8064" x2="21.5" y2="21.79" width="0.2032" layer="16"/>
 <wire x1="20.6944" y1="34.608" x2="20.69" y2="34.67" width="0.2032" layer="16"/>
 <wire x1="35.7312" y1="15.7104" x2="43.2496" y2="15.7104" width="0.2032" layer="16"/>
-<wire x1="29.432" y1="22.0096" x2="35.7312" y2="15.7104" width="0.2032" layer="16"/>
-<wire x1="23.7424" y1="22.0096" x2="29.432" y2="22.0096" width="0.2032" layer="16"/>
+<wire x1="29.432" y1="22.0096" x2="35.7312" y2="15.7104" width="0.254" layer="16"/>
+<wire x1="23.7424" y1="22.0096" x2="29.432" y2="22.0096" width="0.254" layer="16"/>
 <wire x1="22.7264" y1="23.0256" x2="23.7424" y2="22.0096" width="0.2032" layer="16"/>
 <wire x1="43.2496" y1="15.7104" x2="43.26" y2="15.67" width="0.2032" layer="16"/>
 </signal>
-<signal name="N$3">
+<signal name="MTR1">
 <contactref element="7" pad="5"/>
 <contactref element="ESCMTR" pad="4"/>
 <wire x1="43.3004" y1="23.2796" x2="43.26" y2="23.29" width="0.1524" layer="1"/>
-<wire x1="48.736" y1="23.2288" x2="43.4528" y2="23.2288" width="0.2032" layer="1"/>
+<wire x1="48.736" y1="23.2288" x2="43.4528" y2="23.2288" width="0.762" layer="1"/>
 <wire x1="43.4528" y1="23.2288" x2="43.26" y2="23.29" width="0.2032" layer="1"/>
 <wire x1="48.736" y1="23.2288" x2="48.88" y2="23.29" width="0.2032" layer="1"/>
 </signal>
-<signal name="N$6">
+<signal name="MTR2">
 <contactref element="ESCMTR" pad="3"/>
 <contactref element="7" pad="4"/>
 <wire x1="43.3004" y1="25.8704" x2="43.26" y2="25.83" width="0.1524" layer="1"/>
-<wire x1="48.736" y1="25.8704" x2="43.4528" y2="25.8704" width="0.2032" layer="1"/>
+<wire x1="48.736" y1="25.8704" x2="43.4528" y2="25.8704" width="0.762" layer="1"/>
 <wire x1="43.4528" y1="25.8704" x2="43.26" y2="25.83" width="0.2032" layer="1"/>
 <wire x1="48.736" y1="25.8704" x2="48.88" y2="25.83" width="0.2032" layer="1"/>
 </signal>
-<signal name="N$2">
+<signal name="MTR4">
 <contactref element="ESCMTR" pad="1"/>
 <contactref element="7" pad="2"/>
 <wire x1="43.3004" y1="30.8996" x2="43.26" y2="30.91" width="0.1524" layer="1"/>
-<wire x1="48.736" y1="30.9504" x2="43.4528" y2="30.9504" width="0.2032" layer="1"/>
+<wire x1="48.736" y1="30.9504" x2="43.4528" y2="30.9504" width="0.762" layer="1"/>
 <wire x1="43.4528" y1="30.9504" x2="43.26" y2="30.91" width="0.2032" layer="1"/>
 <wire x1="48.736" y1="30.9504" x2="48.88" y2="30.91" width="0.2032" layer="1"/>
 </signal>
-<signal name="N$4">
+<signal name="MTR3">
 <contactref element="ESCMTR" pad="2"/>
 <contactref element="7" pad="3"/>
 <wire x1="43.3004" y1="28.3088" x2="43.26" y2="28.37" width="0.1524" layer="1"/>
-<wire x1="48.736" y1="28.3088" x2="43.4528" y2="28.3088" width="0.2032" layer="1"/>
+<wire x1="48.736" y1="28.3088" x2="43.4528" y2="28.3088" width="0.762" layer="1"/>
 <wire x1="43.4528" y1="28.3088" x2="43.26" y2="28.37" width="0.2032" layer="1"/>
 <wire x1="48.736" y1="28.3088" x2="48.88" y2="28.37" width="0.2032" layer="1"/>
@@
 <contactref element="DSM" pad="1"/>
 <wire x1="21.7424" y1="24.5872" x2="21.5392" y2="24.5872" width="0.2032" layer="1"/>
-<wire x1="28.0416" y1="18.288" x2="21.7424" y2="24.5872" width="0.2032" layer="1"/>
+<wire x1="28.0416" y1="18.288" x2="21.7424" y2="24.5872" width="0.254" layer="1"/>
 <wire x1="21.5392" y1="24.5872" x2="21.5" y2="24.79" width="0.2032" layer="1"/>
 <wire x1="28.0416" y1="18.288" x2="28.21" y2="18.21" width="0.2032" layer="1"/>
